File: EpsilonAnomalain.kicad_pcb (KiCad board)
At the start: 2 copper layers, 48 parts, among them J1 I2C, J2 ServoA, J3 ServoB, J4 ServoC, J5 ServoD, U1 ESP32-S3FN8, U2 ICM-42688-P, U3 BMP388, U4 AHT20, U5 W25N01GVZEIG, U6 KCSA02-105, U7 74HC595

Commit message: rev2.10
Parts:
- removed R11, R12, R13, R14, R15, R16, R17, R18: 1k, Resistor_SMD:R_0402_1005Metric
- added C15: 10uF, Capacitor_SMD:C_0402_1005Metric, F.Cu at (70.9, 88.7)
- added C18: 1uF, Capacitor_SMD:C_0402_1005Metric, F.Cu at (70.9, 90.7)
- added C19: 100nF, Capacitor_SMD:C_0402_1005Metric, F.Cu at (70.9, 92.6)
- added C20: 100nF, Capacitor_SMD:C_0402_1005Metric, F.Cu at (70.9, 94.6)
- added C21: 8.2nF, Capacitor_SMD:C_0402_1005Metric, F.Cu at (70.9, 96.6)
- added C22: 1uF, Capacitor_SMD:C_0402_1005Metric, F.Cu at (73.7, 86.7)
- added C23: 1uF, Capacitor_SMD:C_0402_1005Metric, F.Cu at (73.7, 88.7)
- added C24: 43pF, Capacitor_SMD:C_0402_1005Metric, F.Cu at (73.7, 90.7)
- added C25: 1nF, Capacitor_SMD:C_0402_1005Metric, F.Cu at (73.7, 92.6)
- added C26: 100uF, Capacitor_SMD:C_1206_3216Metric, F.Cu at (103.8, 91.2)
- added C27: 100uF, Capacitor_SMD:C_1206_3216Metric, F.Cu at (103.8, 94.6)
- added C28: 100uF, Capacitor_SMD:C_1206_3216Metric, F.Cu at (114.3, 49.4)
- added C29: 100uF, Capacitor_SMD:C_1206_3216Metric, F.Cu at (121.0, 49.4)
- added C30: 100uF, Capacitor_SMD:C_1206_3216Metric, F.Cu at (127.7, 49.4)
- added C31: 100uF, Capacitor_SMD:C_1206_3216Metric, F.Cu at (134.5, 49.4)
- added C6: 10uF, Capacitor_SMD:C_0402_1005Metric, F.Cu at (70.9, 86.7)
- added D1: BAT54CW, Package_TO_SOT_SMD:SOT-323_SC-70, F.Cu at (71.7, 99.6)
- added D2: DFLS130L, Diode_SMD:D_PowerDI-123, F.Cu at (78.2, 97.5)
- added D3: DFLS130L, Diode_SMD:D_PowerDI-123, F.Cu at (78.2, 101.2)
- added J6: USB_C, Connector_USB:USB_C_Receptacle_GCT_USB4105-xx-A_16P_TopMnt_Horizontal, F.Cu at (81.0, 91.0)
- added L2: 1uH, Capacitor_SMD:C_0402_1005Metric, F.Cu at (73.7, 94.6)
- added R21: 267k, Resistor_SMD:R_0402_1005Metric, F.Cu at (82.7, 103.8)
- added R22: 470k, Resistor_SMD:R_0402_1005Metric, F.Cu at (82.7, 105.8)
- added R23: 118k, Resistor_SMD:R_0402_1005Metric, F.Cu at (82.7, 107.8)
- added R24: 124k, Resistor_SMD:R_0402_1005Metric, F.Cu at (85.6, 103.8)
- added R25: 10k, Resistor_SMD:R_0402_1005Metric, F.Cu at (85.6, 105.8)
- added R26: 100, Resistor_SMD:R_0402_1005Metric, F.Cu at (85.6, 107.8)
- added R27: 124k, Resistor_SMD:R_0402_1005Metric, F.Cu at (88.5, 103.8)
- added R28: 5.1k, Resistor_SMD:R_0402_1005Metric, F.Cu at (88.5, 105.8)
- added R29: 5.1k, Resistor_SMD:R_0402_1005Metric, F.Cu at (88.5, 107.8)
- added RN1: 1k, Resistor_SMD:R_Array_Convex_4x0402, F.Cu at (66.2, 57.4)
- added RN2: 1k, Resistor_SMD:R_Array_Convex_4x0402, F.Cu at (69.3, 57.4)
- added SW1: ON, Button_Switch_SMD:SW_SPST_TL3342, F.Cu at (86.0, 99.2)
- added U10: USBLC6-2SC6, Package_TO_SOT_SMD:SOT-23-6, F.Cu at (83.9, 82.0)
- added U8: TPS61088, UltraLibrarian:RHL0020A, F.Cu at (120.8, 90.4)
- added U9: AP2112K-3.3, Package_TO_SOT_SMD:SOT-23-5, F.Cu at (89.4, 88.1)
- added Y1: 40 MHz, Crystal:Crystal_SMD_3225-4Pin_3.2x2.5mm, F.Cu at (77.8, 105.2)
- C13, C14: value 0.01uF -> 10nF
- C16, C17: value 0.1uF -> 100nF
- U6: value KCSA02-105 -> SS206SURWA/S530-A3/S290; footprint Display_7Segment:KCSC02-105 -> CustomPackage:SS206SURWA
- U7: footprint Package_SO:SO-16_3.9x9.9mm_P1.27mm -> Package_SO:TSSOP-16_4.4x5mm_P0.65mm
- moved J5 37.8 mm to (115.8, 53.5), turned to -90 degrees
- moved J4 27.6 mm to (122.5, 53.5), turned to -90 degrees
- moved J3 17.5 mm to (129.2, 53.5), turned to -90 degrees
- moved J2 7.99 mm to (136.0, 53.5), turned to -90 degrees
Connections:
- C1 pad 1: unconnected-(C1-Pad1) -> Net-(U1-XTAL_P)
- C1 pad 2: unconnected-(C1-Pad2) -> Net-(C1-Pad2)
- C17 pad 1: Net-(C17-Pad1) -> GND
- C2 pad 1: unconnected-(C2-Pad1) -> Net-(U1-XTAL_N)
- C2 pad 2: unconnected-(C2-Pad2) -> Net-(C1-Pad2)
- U1 pad 25: unconnected-(U1-GPIO19/USB_D--Pad25) -> /DN
- U1 pad 26: unconnected-(U1-GPIO20/USB_D+-Pad26) -> /DP
- U1 pad 53: unconnected-(U1-XTAL_N-Pad53) -> Net-(U1-XTAL_N)
- U1 pad 54: unconnected-(U1-XTAL_P-Pad54) -> Net-(U1-XTAL_P)
- U3 pad 3: Net-(C17-Pad1) -> GND
- U3 pad 4: /SDA -> unconnected-(U3-SDI/SDA-Pad4)
Routing:
- net Net-(J6-D--PadA7): track 0.00 -> 8.32 mm
Other:
- board outline added: 55 x 74 mm

Commit message: v2.13
Parts:
- added BZ1: Buzzer, Buzzer_Beeper:MagneticBuzzer_CUI_CMT-8504-100-SMT, F.Cu at (150.2, 112.8)
- added C32: 1uF, Capacitor_SMD:C_0402_1005Metric, F.Cu at (146.0, 101.2)
- added D4: Power, LED_SMD:LED_0402_1005Metric, F.Cu at (143.4, 89.7)
- added D5: TX0, LED_SMD:LED_0402_1005Metric, F.Cu at (143.4, 91.7)
- added D6: RX0, LED_SMD:LED_0402_1005Metric, F.Cu at (143.4, 93.7)
- added D7: Action, LED_SMD:LED_0402_1005Metric, F.Cu at (143.4, 95.7)
- added D8: BAT54C, Package_TO_SOT_SMD:SOT-23, F.Cu at (151.6, 119.8)
- added H1: MountingHole, MountingHole:MountingHole_3.2mm_M3_Pad_Via, F.Cu at (210.0, 65.0)
- added H2: MountingHole, MountingHole:MountingHole_3.2mm_M3_Pad_Via, F.Cu at (165.0, 65.0)
- added H3: MountingHole, MountingHole:MountingHole_3.2mm_M3_Pad_Via, F.Cu at (165.0, 129.0)
- added H4: MountingHole, MountingHole:MountingHole_3.2mm_M3_Pad_Via, F.Cu at (210.0, 129.0)
- added Q1: BC817-40, Package_TO_SOT_SMD:SOT-23, F.Cu at (147.0, 120.7)
- added R11: 5.1k, Resistor_SMD:R_0402_1005Metric, F.Cu at (143.1, 97.7)
- added R12: 5.1k, Resistor_SMD:R_0402_1005Metric, F.Cu at (143.1, 99.7)
- added R13: 470, Resistor_SMD:R_0402_1005Metric, F.Cu at (143.1, 101.6)
- added R14: 470, Resistor_SMD:R_0402_1005Metric, F.Cu at (155.2, 119.3)
- added RN3: 1k, Resistor_SMD:R_Array_Convex_4x0402, F.Cu at (146.1, 98.4)
- added SW2: ON, Button_Switch_SMD:SW_SPST_TL3342, F.Cu at (136.9, 92.2)
- added SW3: ON, Button_Switch_SMD:SW_SPST_TL3342, F.Cu at (136.9, 99.3)
- C10, C11, C3, C4, C9: value 0.1uF -> 100nF
- C7: value 0.01uF -> 10nF
- D1: value BAT54CW -> BAT54C; footprint Package_TO_SOT_SMD:SOT-323_SC-70 -> Package_TO_SOT_SMD:SOT-23
- moved C31 97.3 mm to (204.4, 117.1), turned to -90 degrees
- moved C30 95.7 mm to (195.4, 117.1), turned to -90 degrees
- moved C29 94.1 mm to (186.3, 117.1), turned to -90 degrees
- moved C28 92.4 mm to (177.3, 117.1), turned to -90 degrees
- moved J2 87.8 mm to (200.4, 113.1)
- moved J3 86.1 mm to (191.4, 113.1)
- moved J4 84.4 mm to (182.3, 113.1)
- moved D1 83.6 mm to (151.6, 124.1)
- moved J5 82.8 mm to (173.3, 113.1)
Connections:
- D1 pad 1: Net-(D1-Pad1) -> VDD
- D1 pad 2: VDD -> Net-(D1-Pad2)
- SW1 pad 1: Net-(D1-Pad1) -> Net-(D1-Pad2)
- U1 pad 10: unconnected-(U1-GPIO5-Pad10) -> /VSPI_CLK
- U1 pad 11: unconnected-(U1-GPIO6-Pad11) -> /VSPI_D
- U1 pad 12: unconnected-(U1-GPIO7-Pad12) -> /VSPI_Q
- U1 pad 13: unconnected-(U1-GPIO8-Pad13) -> /VSPI_CS
- U1 pad 23: unconnected-(U1-GPIO17-Pad23) -> /SDA
- U1 pad 24: unconnected-(U1-GPIO18-Pad24) -> /SCL
- U1 pad 27: unconnected-(U1-GPIO21-Pad27) -> /IMU_INT
- U1 pad 38: unconnected-(U1-GPIO33-Pad38) -> /SERVOA
- U1 pad 39: unconnected-(U1-GPIO34-Pad39) -> /SERVOB
- U1 pad 40: unconnected-(U1-GPIO35-Pad40) -> /SERVOC
- U1 pad 41: unconnected-(U1-GPIO36-Pad41) -> /SERVOD
- U1 pad 42: unconnected-(U1-GPIO37-Pad42) -> /SERVOEN
- U1 pad 49: unconnected-(U1-U0TXD-Pad49) -> /TX0_RAW
- U1 pad 50: unconnected-(U1-U0RXD-Pad50) -> /RXD0
- U1 pad 6: unconnected-(U1-GPIO1-Pad6) -> /LD_OE
- U1 pad 7: unconnected-(U1-GPIO2-Pad7) -> /LD_D
- U1 pad 8: unconnected-(U1-GPIO3-Pad8) -> /LD_CLK
- U7 pad 13: GND -> /LD_OE

Commit message: v2.14
Parts:
- removed R1, R2, R3, R4: 100, Resistor_SMD:R_0402_1005Metric
- removed R10, R5, R6, R7, R8, R9: 0, Resistor_SMD:R_0402_1005Metric
- added J7: Power, CustomConnectors:Battery_3V7_Cable_connector_v2, F.Cu at (194.6, 98.8)
- added J8: UART, Connector_JST:JST_XH_B4B-XH-A_1x04_P2.50mm_Vertical, F.Cu at (126.8, 120.3)
- added R15: 5.1k, Resistor_SMD:R_0402_1005Metric, F.Cu at (121.7, 109.5)
- added R16: 5.1k, Resistor_SMD:R_0402_1005Metric, F.Cu at (121.7, 111.5)
- added RN4: 100, Resistor_SMD:R_Array_Convex_4x0402, F.Cu at (109.6, 114.0)
- added RN5: 0, Resistor_SMD:R_Array_Convex_4x0402, F.Cu at (114.4, 118.2)
- added RN6: 0, Resistor_SMD:R_Array_Convex_4x0402, F.Cu at (111.9, 118.2)
- L2: footprint Capacitor_SMD:C_0402_1005Metric -> Inductor_SMD:L_APV_APH0630
- moved C25 85.7 mm to (155.8, 67.7), turned to -90 degrees
- moved R22 84.4 mm to (158.2, 68.2), turned to 180 degrees
- moved R23 84.2 mm to (156.8, 67.8), turned to 90 degrees
- moved C24 83.9 mm to (154.2, 67.2), turned to 180 degrees
- moved C21 81.4 mm to (148.8, 73.3), turned to 90 degrees
- moved C18 80.1 mm to (147.2, 66.2), turned to 90 degrees
- moved C20 79.9 mm to (147.2, 70.8), turned to 90 degrees
- moved C19 78.8 mm to (147.3, 73.3), turned to -90 degrees
- moved R24 76.6 mm to (152.8, 67.0), turned to 90 degrees
- moved R27 74.7 mm to (154.2, 68.2)
- moved R21 73.5 mm to (147.2, 68.5), turned to 90 degrees
- moved L2 72.4 mm to (141.5, 69.0)
- moved C27 55.9 mm to (154.8, 71.7), turned to -90 degrees
- moved U5 54.0 mm to (115.2, 122.6), turned to 180 degrees
- moved C26 40.3 mm to (140.2, 74.0)
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Connections:
- U1 pad 43: unconnected-(U1-GPIO38-Pad43) -> /BUZ
- U1 pad 44: unconnected-(U1-MTCK-Pad44) -> /Action
- U1 pad 9: unconnected-(U1-GPIO4-Pad9) -> /V_ADC
- U3 pad 4: unconnected-(U3-SDI/SDA-Pad4) -> /SDA
Routing:
- net Net-(RN5-R1.1): track 0.00 -> 8.29 mm
- net Net-(RN5-R2.1): track 0.00 -> 6.82 mm
- net Net-(U8-FB): track 0.00 -> 6.50 mm
- net Net-(RN6-R4.2): track 0.00 -> 4.93 mm
- net GND: track 0.00 -> 4.32 mm
- net Net-(RN6-R1.2): track 0.00 -> 3.77 mm
- net Net-(U8-COMP): track 0.00 -> 3.31 mm
- net Net-(U8-VCC): track 0.00 -> 2.67 mm
- net /FSPI_HD: track 0.00 -> 2.46 mm
- net Net-(C20-Pad2): track 0.00 -> 2.29 mm
- net Net-(RN6-R2.2): track 0.00 -> 2.29 mm
- net /FSPI_CS0: track 0.00 -> 1.76 mm
- net /FSPI_WP: track 0.00 -> 1.72 mm
- net /FSPI_D: track 0.00 -> 1.72 mm
- net /FSPI_Q: track 0.00 -> 1.67 mm
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- added copper zone on F.Cu, net GND

Commit message: v2.16
Parts:
- removed RN4: 100, Resistor_SMD:R_Array_Convex_4x0402
- added C33: 1uF, Capacitor_SMD:C_0402_1005Metric, F.Cu at (232.9, 112.5)
- added R1: 10k, Resistor_SMD:R_0402_1005Metric, F.Cu at (258.0, 96.4)
- added R2: 10k, Resistor_SMD:R_0402_1005Metric, F.Cu at (266.7, 112.5)
- added REF**: Linkkalu_v1_8.0x8.4mm, Logos:Linkkalu_v1_8.0x8.4mm, F.Cu at (241.0, 79.0)
- added RN8: R_Pack04_Split, Resistor_SMD:R_Array_Convex_4x0402, F.Cu at (259.7, 98.5)
- D4, D5, D6, D7: footprint LED_SMD:LED_0402_1005Metric -> LED_SMD:LED_0603_1608Metric
- J1: footprint Connector_JST:JST_XH_B4B-XH-A_1x04_P2.50mm_Vertical -> Connector_JST:JST_GH_SM04B-GHS-TB_1x04-1MP_P1.25mm_Horizontal
- R11, R12: value 5.1k -> 10k
- moved D3 201.0 mm to (279.1, 97.7)
- moved C23 199.6 mm to (273.2, 95.2), turned to -90 degrees
- moved J6 198.7 mm to (279.3, 104.5), turned to 90 degrees
- moved C22 197.5 mm to (270.9, 98.0), turned to 90 degrees
- moved D2 195.7 mm to (273.9, 97.7), turned to 180 degrees
- moved SW1 192.2 mm to (278.1, 93.3)
- moved C11 189.9 mm to (268.4, 103.8), turned to -90 degrees
- moved RN1 189.6 mm to (249.7, 105.5)
- moved C2 189.4 mm to (266.1, 92.3), turned to -90 degrees
- moved U10 189.2 mm to (271.8, 104.5), turned to 180 degrees
- moved C12 188.7 mm to (267.5, 103.8), turned to -90 degrees
- moved C10 188.2 mm to (266.4, 103.8), turned to -90 degrees
- moved C9 187.6 mm to (267.2, 92.3), turned to 90 degrees
- moved RN2 187.4 mm to (249.7, 108.0)
- moved C6 187.4 mm to (258.0, 95.5)
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Connections:
- C1 pad 2: Net-(C1-Pad2) -> GND
- C2 pad 2: Net-(C1-Pad2) -> GND
- J1 pad 1: VDD -> /SDA
- J1 pad 2: GND -> /SCL
- J1 pad 3: /SCL -> GND
- J1 pad 4: /SDA -> VDD
- U1 pad 10: /VSPI_CLK -> /VSPI_CS
- U1 pad 11: /VSPI_D -> /IMU_INT
- U1 pad 12: /VSPI_Q -> /V_ADC
- U1 pad 13: /VSPI_CS -> unconnected-(U1-GPIO8-Pad13)
- U1 pad 27: /IMU_INT -> unconnected-(U1-GPIO21-Pad27)
- U1 pad 6: /LD_OE -> /VSPI_Q
- U1 pad 7: /LD_D -> /VSPI_D
- U1 pad 8: /LD_CLK -> unconnected-(U1-GPIO3-Pad8)
- U1 pad 9: /V_ADC -> /VSPI_CLK
- Y1 pad 2: Net-(C1-Pad2) -> GND
- Y1 pad 4: Net-(C1-Pad2) -> GND
Routing:
- net GND: track 4.32 -> 104.6 mm, vias 0 -> 28
- net +6V: track 0.00 -> 67.1 mm
- net +3V8: track 0.00 -> 52.7 mm, vias 0 -> 10
- net /RXD0: track 0.00 -> 40.8 mm, vias 0 -> 2
- net /TX0_RAW: track 0.00 -> 35.6 mm, vias 0 -> 3
- net VDD: track 0.00 -> 30.0 mm, vias 0 -> 9
- net Net-(D2-K): track 0.00 -> 19.3 mm
- net Net-(RN6-R3.2): track 0.00 -> 17.5 mm
- net /CHIP_PU: track 0.00 -> 15.4 mm, vias 0 -> 1
- net Net-(RN2-R3.1): track 0.00 -> 13.4 mm, vias 0 -> 2
- net Net-(BZ1--): track 0.00 -> 13.2 mm
- net Net-(D2-A): track 0.00 -> 12.3 mm, vias 0 -> 2
- net Net-(RN2-R2.1): track 0.00 -> 11.8 mm, vias 0 -> 2
- net Net-(J6-CC2): track 0.00 -> 11.8 mm
- net Net-(RN2-R4.1): track 0.00 -> 11.0 mm
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- added copper zone on F.Cu, net +6V
- added copper zone on In1.Cu, net GND
- added copper zone on F.Cu, net Net-(C20-Pad2)
Other:
- board size 55 x 74 mm -> 55 x 55 mm
- copper layers 2 -> 4
- board text added: "A"
- board text added: "ACT"
- board text added: "B"
- board text added: "BOOT"
- board text added: "C"
- board text added: "D"
- board text added: "EpsilonAnomalain"
- board text added: "PWR"
- board text added: "RES"
- board text added: "RXD"
- board text added: "TXD"
- board text added: "TXD RXD GND 3V3"

Commit message: v2.20
Parts:
- removed R20, R28, R29: 5.1k, Resistor_SMD:R_0402_1005Metric
- removed R21: 267k, Resistor_SMD:R_0402_1005Metric
- removed R22: 470k, Resistor_SMD:R_0402_1005Metric
- removed R23: 118k, Resistor_SMD:R_0402_1005Metric
- removed R24, R27: 124k, Resistor_SMD:R_0402_1005Metric
- removed R25: 10k, Resistor_SMD:R_0402_1005Metric
- removed R26: 100, Resistor_SMD:R_0402_1005Metric
- removed RN8: R_Pack04_Split, Resistor_SMD:R_Array_Convex_4x0402
- added C34: 100nF, Capacitor_SMD:C_0402_1005Metric, F.Cu at (258.6, 110.0)
- added G***: LOGO, Logos:OKB_Iva_v2_9.3x8mm, F.Cu at (242.3, 79.0)
- added R1: 470k, Resistor_SMD:R_0402_1005Metric, F.Cu at (236.1, 117.6)
- added R12: 5.1k, Resistor_SMD:R_0402_1005Metric, F.Cu at (258.3, 91.3)
- added R2: 267k, Resistor_SMD:R_0402_1005Metric, F.Cu at (235.4, 107.1)
- added R3: 118k, Resistor_SMD:R_0402_1005Metric, F.Cu at (236.1, 116.6)
- added R4: 100, Resistor_SMD:R_0402_1005Metric, F.Cu at (271.7, 94.7)
- added R5: 28.7k, Resistor_SMD:R_0402_1005Metric, F.Cu at (235.6, 114.2)
- added R6: 10k, Resistor_SMD:R_0402_1005Metric, F.Cu at (271.7, 95.7)
- added R7: 124k, Resistor_SMD:R_0402_1005Metric, F.Cu at (236.9, 112.6)
- added R8: 5.1k, Resistor_SMD:R_0402_1005Metric, F.Cu at (273.8, 108.7)
- added R9: 5.1k, Resistor_SMD:R_0402_1005Metric, F.Cu at (272.9, 107.1)
- added RN1: R_Pack04_Split, Resistor_SMD:R_Array_Convex_4x0402, F.Cu at (259.7, 98.5)
- moved REF** 11.2 mm to (252.2, 78.9)
- moved J8 5.16 mm to (229.7, 94.5)
- moved C9 4.54 mm to (231.0, 96.0), turned to 180 degrees
- moved R18 2.79 mm to (259.5, 101.7)
- moved R19 0.69 mm to (258.5, 101.7), turned to -90 degrees
- moved C19 0.18 mm to (237.5, 107.0)
- moved C17 0.05 mm to (231.1, 107.1)
- renumbered C20 to C1, C8 to C10, C7 to C11, C23 to C12, C25 to C13, C27 to C14, C9 to C15, C22 to C16, C19 to C17, C24 to C18, C18 to C19, C6 to C2, C21 to C20, C16 to C21, C14 to C22, C15 to C23, C13 to C24, C17 to C25, C28 to C26, C1 to C27, C2 to C28, C5 to C3, C33 to C32, C32 to C33, C3 to C5, C11 to C6, C12 to C7, C10 to C8, C26 to C9, D2 to D1, D3 to D2, D1 to D3, D8 to D4, D4 to D5, D5 to D6, D6 to D7, D7 to D8, H3 to H2, H2 to H3, J6 to J1, J1 to J2, J2 to J3, J3 to J4, J4 to J5, J5 to J6, J8 to J7, J7 to J8, R1 to R10, R19 to R11, R11 to R15, R12 to R16, R2 to R17, R15 to R18, R16 to R19, RN3 to RN2, RN6 to RN3, RN1 to RN4, RN2 to RN5, RN5 to RN6, U9 to U1, U5 to U10, U8 to U2, U10 to U3, U1 to U4, U2 to U5, U4 to U6, U3 to U7, U6 to U8, U7 to U9
Connections:
- U4 pad 13: unconnected-(U1-GPIO8-Pad13) -> /LD_CLK
- U4 pad 27: unconnected-(U1-GPIO21-Pad27) -> /BUZ
- U4 pad 28: unconnected-(U1-SPICS1-Pad28) -> /LD_D
- U4 pad 43: /BUZ -> /OFF
- U4 pad 45: unconnected-(U1-MTDO-Pad45) -> /LD_OE
Routing:
- net GND: track 104.6 -> 348.7 mm, vias 28 -> 126
- net VDD: track 30.0 -> 165.4 mm, vias 9 -> 16
- net +3V8: track 52.7 -> 135.3 mm, vias 10 -> 19
- net /SERVOEN: track 0.00 -> 47.0 mm, vias 0 -> 2
- net /LD_OE: track 0.00 -> 44.6 mm, vias 0 -> 2
- net /SERVOD: track 0.00 -> 42.3 mm, vias 0 -> 2
- net /SERVOC: track 0.00 -> 35.1 mm, vias 0 -> 2
- net /SCL: track 6.52 -> 38.3 mm, vias 2 -> 4
- net /SDA: track 5.33 -> 36.4 mm, vias 0 -> 2
- net /SERVOB: track 0.00 -> 28.5 mm, vias 0 -> 2
- net /LD_D: track 0.00 -> 25.7 mm, vias 0 -> 2
- net /SERVOA: track 0.00 -> 25.1 mm, vias 0 -> 2
- net /LD_CLK: track 0.00 -> 17.4 mm
- net /CHIP_PU: track 15.4 -> 30.1 mm, vias 1 -> 2
- net /BOOT: track 9.08 -> 20.7 mm, vias 1 -> 2
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- added copper zone on B.Cu, net +3V8
- added copper zone on F.Cu, net +3V8
- added copper zone on B.Cu, net GND
- added copper zone on F.Cu, net VDD
- added copper zone on In2.Cu, net VDD
Other:
- board text added: "30.11.2024 v2.20"
- board text added: "3V7"
- board text added: "GND"
- board text added: "I2C"
- board text added: "R"
- board text added: "X"
- board text added: "Y"
- board text added: "Z"
- board text removed: "BOOT"
- board text removed: "RES"

Commit message: v2.22
Parts:
- BZ1: value Buzzer -> CMT-8504-100
- L1: value 2.7nH -> 2.2nH
- RN1: value R_Pack04_Split -> 47
- SW1, SW2, SW3: value ON -> TS-1187A-B-A-B
- U7: footprint CustomPackage:BMP388 -> CustomPackage:BMP388_v2
Routing:
- net GND: track 348.7 -> 344.1 mm, vias 126 -> 131
- net /SCL: track 38.3 -> 37.7 mm
Other:
- board text added: "12.12.2024 v2.22"
- board text removed: "30.11.2024 v2.20"

Commit message: Update
Parts:
- moved R10 0.49 mm to (257.5, 96.4)
Routing:
- net GND: track 344.1 -> 339.9 mm, vias 131 -> 148
- net /LD_OE: track 44.6 -> 45.5 mm
- net /DP: track 6.21 -> 7.02 mm
- net VDD: track 165.4 -> 164.7 mm, vias 16 -> 21

Commit message: update
Parts:
- moved C14 53.0 mm to (193.2, 78.6)
- moved C18 53.0 mm to (197.4, 78.6)
- moved D1 53.0 mm to (234.7, 62.1)
- moved G*** 53.0 mm to (203.1, 43.4)
- moved J5 53.0 mm to (208.7, 82.3)
- moved J8 53.0 mm to (190.5, 58.9)
- moved L1 53.0 mm to (220.7, 60.2)
- moved R11 53.0 mm to (219.1, 56.7)
- moved R8 53.0 mm to (234.6, 73.1)
- moved REF** 53.0 mm to (213.0, 43.3)
- moved SW2 53.0 mm to (204.6, 58.4)
- moved SW3 53.0 mm to (210.6, 58.4)
- moved U10 53.0 mm to (224.6, 72.5)
- moved C17 53.0 mm to (191.9, 71.5)
- moved C19 53.0 mm to (198.3, 71.5)
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