File: EpsilonAnomalain.kicad_pcb (KiCad board)
At the start: 4 copper layers, 55 x 55 mm, 99 parts, among them J1 USB_C, J2 I2C, J3 ServoA, J4 ServoB, J5 ServoC, J6 ServoD, J7 UART, J8 Power, Q1 BC817-40, SW1 TS-1187A-B-A-B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

Commit message: dimentions added
Other:
- board text added: "2.5"
- board text added: "3.2"
